File: PCB/L298N_DRIVER.kicad_pcb (KiCad board)
At the start: 2 copper layers, 59.5 x 43.5 mm, 21 parts, among them J1 PWM-INPUT, J2 MOT-OUTPUT, J3 +5V, J4 +BATT, J5 SERIAL, J6 I2C, U1 L298N, U2 adino2

Commit message: pcb update
Parts:
- added J7: MOT02, Connector_JST:JST_PH_S2B-PH-K_1x02_P2.00mm_Horizontal, F.Cu at (177.4, 70.7)
- added J8: PWM-B, Connector_JST:JST_PH_S3B-PH-K_1x03_P2.00mm_Horizontal, F.Cu at (125.3, 73.3)
- J1: value PWM-INPUT -> PWM-A; footprint Connector_JST:JST_PH_S4B-PH-K_1x04_P2.00mm_Horizontal -> Connector_JST:JST_PH_S3B-PH-K_1x03_P2.00mm_Horizontal
- J2: value MOT-OUTPUT -> MOT1; footprint Connector_JST:JST_PH_S4B-PH-K_1x04_P2.00mm_Horizontal -> Connector_JST:JST_PH_S2B-PH-K_1x02_P2.00mm_Horizontal
- J5, J6: footprint Connector_JST:JST_PH_S4B-PH-K_1x04_P2.00mm_Horizontal -> Connector_JST:JST_PH_B4B-PH-K_1x04_P2.00mm_Vertical
- moved J6 44.7 mm to (129.8, 59.5)
- moved J4 43.8 mm to (174.5, 56.3), turned to 90 degrees
- moved J1 7.81 mm to (125.3, 64.5)
- moved J2 7.57 mm to (177.4, 63.9)
- moved J5 5.43 mm to (122.7, 59.6), turned to 90 degrees
- moved H2 3.23 mm to (180.2, 47.6)
- moved H1 3.10 mm to (180.1, 83.8)
- moved J3 2.93 mm to (177.4, 77.7)
- moved H3 2.82 mm to (122.7, 48.1)
- moved U2 2.67 mm to (149.0, 79.8)
- moved H4 2.54 mm to (122.9, 83.5)
- moved D2 0.41 mm to (161.6, 67.0)
Connections:
- J1 pad 3: /PWM_B -> GND
Other:
- board size 59.5 x 43.5 mm -> 64.8 x 43.5 mm
- board text added: "L298N DRIVER VER1.1"
- board text removed: "L298N DRIVER VER1.0"

Commit message: v1.1
Parts:
- moved D2 18.4 mm to (145.9, 57.4), turned to 180 degrees
- moved C1 18.2 mm to (166.4, 50.8), turned to 90 degrees
- moved D6 17.2 mm to (145.9, 64.5), turned to 180 degrees
- moved D8 16.3 mm to (145.9, 68.1), turned to 180 degrees
- moved D4 15.7 mm to (145.9, 61.0), turned to 180 degrees
- moved D7 15.5 mm to (155.6, 68.1), turned to 180 degrees
- moved D5 15.5 mm to (155.5, 64.5), turned to 180 degrees
- moved D3 15.5 mm to (155.5, 61.0), turned to 180 degrees
- moved D1 15.5 mm to (155.5, 57.4), turned to 180 degrees
- moved U1 1.53 mm to (141.0, 54.1)
Other:
- net class MOT added: clearance 0.2, trace_width 1, via_dia 0.8, via_drill 0.4
Changed lines of the file:
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@@
     (add_net /IN3)
     (add_net /IN4)
-    (add_net /OUT1)
-    (add_net /OUT2)
-    (add_net /OUT3)
-    (add_net /OUT4)
     (add_net /PWM_A)
     (add_net /PWM_B)
@@
     (uvia_drill 0.1)
     (add_net +BATT)
+  )
+  (net_class MOT ""
+    (clearance 0.2)
+    (trace_width 1)
+    (via_dia 0.8)
+    (via_drill 0.4)
+    (uvia_dia 0.3)
+    (uvia_drill 0.1)
+    (add_net /OUT1)
+    (add_net /OUT2)
+    (add_net /OUT3)
+    (add_net /OUT4)
   )
   (module Connector_JST:JST_PH_S3B-PH-K_1x03_P2.00mm_Horizontal (layer F.Cu)
@@
   )
   (module 1N4007:DIOM5327X242N (layer F.Cu)
-    (at 161.6358 64.0334)
+    (at 145.882 68.072 180)
     (descr "sma do-214ac")
     (tags Diode)
@@
       (effects (font (size 1.27 1.27) (thickness 0.254)))
     )
-    (pad 2 smd rect (at 2.2 0 90) (size 2.15 2.3) (layers F.Cu F.Paste F.Mask)
+    (pad 2 smd rect (at 2.2 0 270) (size 2.15 2.3) (layers F.Cu F.Paste F.Mask)
       (net 3 GND))
-    (pad 1 smd rect (at -2.2 0 90) (size 2.15 2.3) (layers F.Cu F.Paste F.Mask)
+    (pad 1 smd rect (at -2.2 0 270) (size 2.15 2.3) (layers F.Cu F.Paste F.Mask)
       (net 6 /OUT4))
     (model 1N4007.stp
@@
   )
   (module 1N4007:DIOM5327X242N (layer F.Cu)
-    (at 140.122 67.31)
+    (at 155.616 68.072 180)
     (descr "sma do-214ac")
     (tags Diode)
@@
       (effects (font (size 1.27 1.27) (thickness 0.254)))
     )
-    (pad 2 smd rect (at 2.2 0 90) (size 2.15 2.3) (layers F.Cu F.Paste F.Mask)
+    (pad 2 smd rect (at 2.2 0 270) (size 2.15 2.3) (layers F.Cu F.Paste F.Mask)
       (net 6 /OUT4))
-    (pad 1 smd rect (at -2.2 0 90) (size 2.15 2.3) (layers F.Cu F.Paste F.Mask)
+    (pad 1 smd rect (at -2.2 0 270) (size 2.15 2.3) (layers F.Cu F.Paste F.Mask)
       (net 2 +BATT))
     (model 1N4007.stp
@@
   )
   (module 1N4007:DIOM5327X242N (layer F.Cu)
-    (at 161.63 57.658)
+    (at 145.882 64.516 180)
     (descr "sma do-214ac")
     (tags Diode)
@@
       (effects (font (size 1.27 1.27) (thickness 0.254)))
     )
-    (pad 2 smd rect (at 2.2 0 90) (size 2.15 2.3) (layers F.Cu F.Paste F.Mask)
+    (pad 2 smd rect (at 2.2 0 270) (size 2.15 2.3) (layers F.Cu F.Paste F.Mask)
       (net 3 GND))
-    (pad 1 smd rect (at -2.2 0 90) (size 2.15 2.3) (layers F.Cu F.Paste F.Mask)
+    (pad 1 smd rect (at -2.2 0 270) (size 2.15 2.3) (layers F.Cu F.Paste F.Mask)
       (net 5 /OUT3))
     (model 1N4007.stp
@@
   )
   (module 1N4007:DIOM5327X242N (layer F.Cu)
-    (at 140.04 64.008)
+    (at 155.534 64.516 180)
     (descr "sma do-214ac")
     (tags Diode)
@@
       (effects (font (size 1.27 1.27) (thickness 0.254)))
     )
-    (pad 2 smd rect (at 2.2 0 90) (size 2.15 2.3) (layers F.Cu F.Paste F.Mask)
+    (pad 2 smd rect (at 2.2 0 270) (size 2.15 2.3) (layers F.Cu F.Paste F.Mask)
       (net 5 /OUT3))
-    (pad 1 smd rect (at -2.2 0 90) (size 2.15 2.3) (layers F.Cu F.Paste F.Mask)
+    (pad 1 smd rect (at -2.2 0 270) (size 2.15 2.3) (layers F.Cu F.Paste F.Mask)
       (net 2 +BATT))
     (model 1N4007.stp
@@
   )
   (module 1N4007:DIOM5327X242N (layer F.Cu)
-    (at 161.63 60.96)
+    (at 145.882 60.96 180)
     (descr "sma do-214ac")
     (tags Diode)
@@
       (effects (font (size 1.27 1.27) (thickness 0.254)))
     )
-    (pad 2 smd rect (at 2.2 0 90) (size 2.15 2.3) (layers F.Cu F.Paste F.Mask)
+    (pad 2 smd rect (at 2.2 0 270) (size 2.15 2.3) (layers F.Cu F.Paste F.Mask)
       (net 3 GND))
-    (pad 1 smd rect (at -2.2 0 90) (size 2.15 2.3) (layers F.Cu F.Paste F.Mask)
+    (pad 1 smd rect (at -2.2 0 270) (size 2.15 2.3) (layers F.Cu F.Paste F.Mask)
       (net 4 /OUT2))
     (model 1N4007.stp
@@
   )
   (module 1N4007:DIOM5327X242N (layer F.Cu)
-    (at 140.04 60.706)
+    (at 155.534 60.96 180)
     (descr "sma do-214ac")
     (tags Diode)
@@
       (effects (font (size 1.27 1.27) (thickness 0.254)))
     )
-    (pad 2 smd rect (at 2.2 0 90) (size 2.15 2.3) (layers F.Cu F.Paste F.Mask)
+    (pad 2 smd rect (at 2.2 0 270) (size 2.15 2.3) (layers F.Cu F.Paste F.Mask)
       (net 4 /OUT2))
-    (pad 1 smd rect (at -2.2 0 90) (size 2.15 2.3) (layers F.Cu F.Paste F.Mask)
+    (pad 1 smd rect (at -2.2 0 270) (size 2.15 2.3) (layers F.Cu F.Paste F.Mask)
       (net 2 +BATT))
     (model 1N4007.stp
@@
   )
   (module 1N4007:DIOM5327X242N (layer F.Cu)
-    (at 161.6104 67.0052)
+    (at 145.882 57.404 180)
     (descr "sma do-214ac")
     (tags Diode)
@@
       (effects (font (size 1.27 1.27) (thickness 0.254)))
     )
-    (fp_text value D_ALT (at 0 0) (layer F.SilkS) hide
+    (fp_text value D_ALT (at 0.594 0) (layer F.SilkS) hide
       (effects (font (size 1.27 1.27) (thickness 0.254)))
     )
@@
       (effects (font (size 1.27 1.27) (thickness 0.254)))
     )
-    (pad 2 smd rect (at 2.2 0 90) (size 2.15 2.3) (layers F.Cu F.Paste F.Mask)
+    (pad 2 smd rect (at 2.2 0 270) (size 2.15 2.3) (layers F.Cu F.Paste F.Mask)
       (net 3 GND))
-    (pad 1 smd rect (at -2.2 0 90) (size 2.15 2.3) (layers F.Cu F.Paste F.Mask)
+    (pad 1 smd rect (at -2.2 0 270) (size 2.15 2.3) (layers F.Cu F.Paste F.Mask)
       (net 1 /OUT1))
     (model 1N4007.stp
@@
   )
   (module 1N4007:DIOM5327X242N (layer F.Cu)
-    (at 140.04 57.404)
+    (at 155.534 57.404 180)
     (descr "sma do-214ac")
     (tags Diode)
@@
       (effects (font (size 1.27 1.27) (thickness 0.254)))
     )
-    (pad 2 smd rect (at 2.2 0 90) (size 2.15 2.3) (layers F.Cu F.Paste F.Mask)
+    (pad 2 smd rect (at 2.2 0 270) (size 2.15 2.3) (layers F.Cu F.Paste F.Mask)
       (net 1 /OUT1))
-    (pad 1 smd rect (at -2.2 0 90) (size 2.15 2.3) (layers F.Cu F.Paste F.Mask)
+    (pad 1 smd rect (at -2.2 0 270) (size 2.15 2.3) (layers F.Cu F.Paste F.Mask)
       (net 2 +BATT))
     (model 1N4007.stp
@@
   )
   (module Capacitor_SMD:C_Elec_8x10.2 (layer F.Cu)
-    (at 151.594 61.468 180)
+    (at 166.37 50.844 90)
     (descr "SMD capacitor, aluminum electrolytic nonpolar, 8.0x10.2mm")
     (tags "capacitor electrolyic nonpolar")
     (attr smd)
-    (fp_text reference C1 (at 0 -5.2) (layer F.SilkS)
-      (effects (font (size 1 1) (thickness 0.15)))
-    )
-    (fp_text value C_Small (at 0 5.2) (layer F.Fab) hide
-      (effects (font (size 1 1) (thickness 0.15)))
-    )
-    (fp_text user %R (at 0 0) (layer F.Fab)
+    (fp_text reference C1 (at 0 -5.2 90) (layer F.SilkS)
+      (effects (font (size 1 1) (thickness 0.15)))
+    )
+    (fp_text value C_Small (at 0 5.2 90) (layer F.Fab) hide
+      (effects (font (size 1 1) (thickness 0.15)))
+    )
+    (fp_text user %R (at 0 0 90) (layer F.Fab)
       (effects (font (size 1 1) (thickness 0.15)))
     )
@@
     (fp_line (start 4.15 -4.15) (end 4.15 4.15) (layer F.Fab) (width 0.1))
     (fp_circle (center 0 0) (end 4 0) (layer F.Fab) (width 0.1))
-    (pad 2 smd roundrect (at 3.6 0 180) (size 4.5 2.1) (layers F.Cu F.Paste F.Mask) (roundrect_rratio 0.119048)
+    (pad 2 smd roundrect (at 3.6 0 90) (size 4.5 2.1) (layers F.Cu F.Paste F.Mask) (roundrect_rratio 0.119048)
       (net 3 GND))
-    (pad 1 smd roundrect (at -3.6 0 180) (size 4.5 2.1) (layers F.Cu F.Paste F.Mask) (roundrect_rratio 0.119048)
+    (pad 1 smd roundrect (at -3.6 0 90) (size 4.5 2.1) (layers F.Cu F.Paste F.Mask) (roundrect_rratio 0.119048)
       (net 2 +BATT))
     (model ${KISYS3DMOD}/Capacitor_SMD.3dshapes/C_Elec_8x10.2.wrl
@@
   )
   (module digikey-footprints:Multiwatt-15 (layer F.Cu)
-    (at 142.5 54.102)
+    (at 140.97 54.102)
     (descr http://www.st.com/content/ccc/resource/technical/document/datasheet/ab/d6/fa/99/84/36/49/ee/CD00000017.pdf/files/CD00000017.pdf/jcr:content/translations/en.CD00000017.pdf)
     (fp_text reference U1 (at 9 -10.82) (layer F.SilkS) hide

Commit message: bug fix
Parts:
- +5V GND: renamed from J3
- +BATT GND: renamed from J4
- moved D2 1.27 mm to (144.6, 57.4)
- moved D4 1.27 mm to (144.6, 61.0)
- moved D6 1.27 mm to (144.6, 64.5)
- moved D8 1.27 mm to (144.6, 68.1)
- moved H3 0.66 mm to (122.5, 47.5)
- moved H4 0.46 mm to (123.3, 83.2)
- moved H2 0.31 mm to (180.5, 47.5)
- moved H1 0.20 mm to (180.0, 84.0)
- renumbered J6 to I2C, J2 to MOT1, J7 to MOT2, J1 to PWM-A, J8 to PWM-B, J5 to SERIAL
Routing:
- net GND: track 0.00 -> 204.0 mm, vias 0 -> 1
- net +5V: track 0.00 -> 110.0 mm
- net /OUT1: track 0.00 -> 68.8 mm
- net /SCL: track 0.00 -> 65.4 mm
- net /SDA: track 0.00 -> 62.9 mm
- net /OUT4: track 0.00 -> 61.9 mm
- net +BATT: track 0.00 -> 56.9 mm
- net /OUT2: track 0.00 -> 55.3 mm, vias 0 -> 3
- net /TX: track 0.00 -> 49.5 mm
- net /EN_A: track 0.00 -> 48.1 mm
- net /RX: track 0.00 -> 48.0 mm
- net /OUT3: track 0.00 -> 46.9 mm
- net /EN_B: track 0.00 -> 46.8 mm
- net /IN4: track 0.00 -> 42.5 mm
- net /PWM_A: track 0.00 -> 41.3 mm
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- added copper zone on B.Cu, net GND
- added copper zone on F.Cu, net GND
Other:
- board size 64.8 x 43.5 mm -> 65 x 43.5 mm
